File: brooderCircuit/brooder-mainboard/brooder-mainboard.sch (KiCad schematic (older format))
At the start: 29 parts, among them Q1 BC548, Q2 BT136-500, Q3 BC548, T1 240V to 12V, U1 L7805, U2 MOC3043M

Commit message: first commit
Parts:
- gave numbers to parts that had none: 3
Changed lines of the file:
@@
 SPK
 $Comp
-L Device:Q_NPN_CBE Q?
+L Device:Q_NPN_CBE Q4
 U 1 1 62EA5BB3
 P 9700 1950
-F 0 "Q?" H 9891 1996 50  0000 L CNN
+F 0 "Q4" H 9891 1996 50  0000 L CNN
 F 1 "BC548" H 9891 1905 50  0000 L CNN
 F 2 "" H 9900 2050 50  0001 C CNN
@@
 $EndComp
 $Comp
-L power:+5V #PWR?
+L power:+5V #PWR08
 U 1 1 62EA5BB9
 P 9800 850
-F 0 "#PWR?" H 9800 700 50  0001 C CNN
+F 0 "#PWR08" H 9800 700 50  0001 C CNN
 F 1 "+5V" H 9815 1023 50  0000 C CNN
 F 2 "" H 9800 850 50  0001 C CNN
@@
 $EndComp
 $Comp
-L Device:R R?
+L Device:R R9
 U 1 1 62EA5BBF
 P 9200 1950
-F 0 "R?" V 8993 1950 50  0000 C CNN
+F 0 "R9" V 8993 1950 50  0000 C CNN
 F 1 "330R" V 9084 1950 50  0000 C CNN
 F 2 "" V 9130 1950 50  0001 C CNN
@@
 $EndComp
 $Comp
-L power:GND #PWR?
+L power:GND #PWR09
 U 1 1 62EA5BC5
 P 9800 2250
-F 0 "#PWR?" H 9800 2000 50  0001 C CNN
+F 0 "#PWR09" H 9800 2000 50  0001 C CNN
 F 1 "GND" H 9805 2077 50  0000 C CNN
 F 2 "" H 9800 2250 50  0001 C CNN
@@
 	9800 850  9800 1000
 $Comp
-L Device:R R?
+L Device:R R10
 U 1 1 62EAC17E
 P 9800 1400
-F 0 "R?" H 9870 1446 50  0000 L CNN
+F 0 "R10" H 9870 1446 50  0000 L CNN
 F 1 "30R" H 9870 1355 50  0000 L CNN
 F 2 "" V 9730 1400 50  0001 C CNN

Commit message: add flyback diodes
Parts:
- added D5, D6: D, symbol Device:D
Connections:
- net FAN-: now also D5.1 (K)
- net GND: now also D5.2 (A), D6.2 (A)
- net at Q4.1 (C), R10.2: now also D6.1 (K)
Changed lines of the file:
@@
 $EndComp
 Wire Wire Line
-	7900 1750 7900 1850
+	7900 1750 7900 1800
 Wire Wire Line
 	7000 1550 7150 1550
@@
 FAN-
 Wire Wire Line
-	7900 1350 7900 1150
+	7900 1350 7900 1250
 Wire Wire Line
 	7900 850  7900 1000
@@
 $EndComp
 Wire Wire Line
-	9800 2150 9800 2250
+	9800 2150 9800 2200
 Wire Wire Line
 	8900 1950 9050 1950
@@
 SPK-
 Wire Wire Line
-	9800 1750 9800 1550
+	9800 1750 9800 1650
 Wire Wire Line
 	9800 850  9800 1000
@@
 Wire Wire Line
 	9800 1250 9800 1150
+$Comp
+L Device:D D5
+U 1 1 62DFD53F
+P 8350 1400
+F 0 "D5" V 8396 1320 50  0000 R CNN
+F 1 "D" V 8305 1320 50  0000 R CNN
+F 2 "" H 8350 1400 50  0001 C CNN
+F 3 "~" H 8350 1400 50  0001 C CNN
+	1    8350 1400
+	0    1    1    0
+$EndComp
+$Comp
+L Device:D D6
+U 1 1 62E02AFE
+P 10350 1800
+F 0 "D6" V 10396 1720 50  0000 R CNN
+F 1 "D" V 10305 1720 50  0000 R CNN
+F 2 "" H 10350 1800 50  0001 C CNN
+F 3 "~" H 10350 1800 50  0001 C CNN
+	1    10350 1800
+	0    1    1    0
+$EndComp
+Wire Wire Line
+	8350 1250 7900 1250
+Connection ~ 7900 1250
+Wire Wire Line
+	7900 1250 7900 1150
+Wire Wire Line
+	8350 1550 8350 1800
+Wire Wire Line
+	8350 1800 7900 1800
+Connection ~ 7900 1800
+Wire Wire Line
+	7900 1800 7900 1850
+Wire Wire Line
+	10350 1950 10350 2200
+Wire Wire Line
+	10350 2200 9800 2200
+Connection ~ 9800 2200
+Wire Wire Line
+	9800 2200 9800 2250
+Wire Wire Line
+	10350 1650 9800 1650
+Connection ~ 9800 1650
+Wire Wire Line
+	9800 1650 9800 1550
 $EndSCHEMATC

Commit message: Circuit updates
Parts:
- removed D3: DIODE, symbol pspice:DIODE
- removed R3: 50K, symbol Device:R
- added R?: 15K, symbol Device:R
- C6: value 0.01uF -> 0.1uF
- R1: value 100K -> 20K
Connections:
- net GND: now also R?.1
- net at D1.2 (A): now also C1.1, R1.2
- net at Q1.2 (B), R1.1: now also R?.2
Other:
- moved on the sheet: C1, Q1, R1, R2
Changed lines of the file:
@@
 $EndComp
-$Comp
-L pspice:DIODE D3
-U 1 1 62DD4BC4
-P 4650 1650
-F 0 "D3" H 4650 1915 50  0000 C CNN
-F 1 "DIODE" H 4650 1824 50  0000 C CNN
-F 2 "" H 4650 1650 50  0001 C CNN
-F 3 "~" H 4650 1650 50  0001 C CNN
-	1    4650 1650
-	1    0    0    -1
-$EndComp
-Wire Wire Line
-	4350 1650 4450 1650
 $Comp
 L Device:R R1
 U 1 1 62DD5AED
-P 5100 1650
-F 0 "R1" V 4893 1650 50  0000 C CNN
-F 1 "100K" V 4984 1650 50  0000 C CNN
-F 2 "" V 5030 1650 50  0001 C CNN
-F 3 "~" H 5100 1650 50  0001 C CNN
-	1    5100 1650
+P 4800 1650
+F 0 "R1" V 4593 1650 50  0000 C CNN
+F 1 "20K" V 4684 1650 50  0000 C CNN
+F 2 "" V 4730 1650 50  0001 C CNN
+F 3 "~" H 4800 1650 50  0001 C CNN
+	1    4800 1650
 	0    1    1    0
 $EndComp
@@
 L Device:CP C1
 U 1 1 62DD6602
-P 4900 1850
-F 0 "C1" H 5018 1896 50  0000 L CNN
-F 1 "2.2uF" H 5018 1805 50  0000 L CNN
-F 2 "" H 4938 1700 50  0001 C CNN
-F 3 "~" H 4900 1850 50  0001 C CNN
-	1    4900 1850
+P 4600 1850
+F 0 "C1" H 4718 1896 50  0000 L CNN
+F 1 "2.2uF" H 4718 1805 50  0000 L CNN
+F 2 "" H 4638 1700 50  0001 C CNN
+F 3 "~" H 4600 1850 50  0001 C CNN
+	1    4600 1850
 	1    0    0    -1
 $EndComp
@@
 L power:GND #PWR01
 U 1 1 62DD72E4
-P 4900 2100
-F 0 "#PWR01" H 4900 1850 50  0001 C CNN
-F 1 "GND" H 4905 1927 50  0000 C CNN
-F 2 "" H 4900 2100 50  0001 C CNN
-F 3 "" H 4900 2100 50  0001 C CNN
-	1    4900 2100
-	1    0    0    -1
-$EndComp
-Wire Wire Line
-	4850 1650 4900 1650
-Wire Wire Line
-	4900 1700 4900 1650
-Connection ~ 4900 1650
-Wire Wire Line
-	4900 1650 4950 1650
-Wire Wire Line
-	4900 2000 4900 2100
+P 4600 2100
+F 0 "#PWR01" H 4600 1850 50  0001 C CNN
+F 1 "GND" H 4605 1927 50  0000 C CNN
+F 2 "" H 4600 2100 50  0001 C CNN
+F 3 "" H 4600 2100 50  0001 C CNN
+	1    4600 2100
+	1    0    0    -1
+$EndComp
+Wire Wire Line
+	4600 1700 4600 1650
+Connection ~ 4600 1650
+Wire Wire Line
+	4600 1650 4650 1650
+Wire Wire Line
+	4600 2000 4600 2100
 $Comp
 L Device:Q_NPN_CBE Q1
 U 1 1 62DDA0F5
-P 5500 1650
-F 0 "Q1" H 5691 1696 50  0000 L CNN
-F 1 "BC548" H 5691 1605 50  0000 L CNN
-F 2 "" H 5700 1750 50  0001 C CNN
-F 3 "~" H 5500 1650 50  0001 C CNN
-	1    5500 1650
-	1    0    0    -1
-$EndComp
-Wire Wire Line
-	5250 1650 5300 1650
-Wire Wire Line
-	5600 1850 5600 2000
-Wire Wire Line
-	5600 2000 5300 2000
-Connection ~ 4900 2000
+P 5350 1650
+F 0 "Q1" H 5541 1696 50  0000 L CNN
+F 1 "BC548" H 5541 1605 50  0000 L CNN
+F 2 "" H 5550 1750 50  0001 C CNN
+F 3 "~" H 5350 1650 50  0001 C CNN
+	1    5350 1650
+	1    0    0    -1
+$EndComp
+Wire Wire Line
+	5450 1850 5450 2000
+Connection ~ 4600 2000
 $Comp
 L Device:CP C2
@@
 L Device:R R2
 U 1 1 62DE4809
-P 5600 1200
-F 0 "R2" H 5670 1246 50  0000 L CNN
-F 1 "10K" H 5670 1155 50  0000 L CNN
-F 2 "" V 5530 1200 50  0001 C CNN
-F 3 "~" H 5600 1200 50  0001 C CNN
-	1    5600 1200
-	1    0    0    -1
-$EndComp
-Wire Wire Line
-	5600 1450 5600 1400
-Wire Wire Line
-	5600 1050 5600 950
+P 5450 1200
+F 0 "R2" H 5520 1246 50  0000 L CNN
+F 1 "10K" H 5520 1155 50  0000 L CNN
+F 2 "" V 5380 1200 50  0001 C CNN
+F 3 "~" H 5450 1200 50  0001 C CNN
+	1    5450 1200
+	1    0    0    -1
+$EndComp
+Wire Wire Line
+	5450 1450 5450 1400
+Wire Wire Line
+	5450 1050 5450 950
 $Comp
 L power:+5V #PWR02
 U 1 1 62DE6021
-P 5600 950
-F 0 "#PWR02" H 5600 800 50  0001 C CNN
-F 1 "+5V" H 5615 1123 50  0000 C CNN
-F 2 "" H 5600 950 50  0001 C CNN
-F 3 "" H 5600 950 50  0001 C CNN
-	1    5600 950
-	1    0    0    -1
-$EndComp
-Wire Wire Line
-	5600 1400 5950 1400
-Connection ~ 5600 1400
-Wire Wire Line
-	5600 1400 5600 1350
-Text GLabel 5950 1400 2    50   Input ~ 0
+P 5450 950
+F 0 "#PWR02" H 5450 800 50  0001 C CNN
+F 1 "+5V" H 5465 1123 50  0000 C CNN
+F 2 "" H 5450 950 50  0001 C CNN
+F 3 "" H 5450 950 50  0001 C CNN
+	1    5450 950
+	1    0    0    -1
+$EndComp
+Wire Wire Line
+	5450 1400 5800 1400
+Connection ~ 5450 1400
+Wire Wire Line
+	5450 1400 5450 1350
+Text GLabel 5800 1400 2    50   Input ~ 0
 V_PWROFF
 $Comp
@@
 Wire Wire Line
 	7050 3200 7100 3200
-$Comp
-L Device:R R3
-U 1 1 62E2819C
-P 5300 1800
-F 0 "R3" H 5230 1754 50  0000 R CNN
-F 1 "50K" H 5230 1845 50  0000 R CNN
-F 2 "" V 5230 1800 50  0001 C CNN
-F 3 "~" H 5300 1800 50  0001 C CNN
-	1    5300 1800
-	-1   0    0    1
-$EndComp
-Connection ~ 5300 1650
-Wire Wire Line
-	5300 1950 5300 2000
-Connection ~ 5300 2000
-Wire Wire Line
-	5300 2000 4900 2000
 $Comp
 L Relay_SolidState:MOC3043M U2
@@
 P 5750 4600
 F 0 "C6" H 5865 4646 50  0000 L CNN
-F 1 "0.01uF" H 5865 4555 50  0000 L CNN
+F 1 "0.1uF" H 5865 4555 50  0000 L CNN
 F 2 "" H 5788 4450 50  0001 C CNN
 F 3 "~" H 5750 4600 50  0001 C CNN
@@
 Wire Wire Line
 	9800 1650 9800 1550
+Wire Wire Line
+	4600 2000 5050 2000
+Wire Wire Line
+	5050 1950 5050 2000
+Wire Wire Line
+	4350 1650 4600 1650
+Wire Wire Line
+	5050 2000 5450 2000
+Connection ~ 5050 2000
+Wire Wire Line
+	4950 1650 5050 1650
+$Comp
+L Device:R R?
+U 1 1 62E44665
+P 5050 1800
+F 0 "R?" V 4843 1800 50  0000 C CNN
+F 1 "15K" V 4934 1800 50  0000 C CNN
+F 2 "" V 4980 1800 50  0001 C CNN
+F 3 "~" H 5050 1800 50  0001 C CNN
+	1    5050 1800
+	-1   0    0    1
+$EndComp
+Connection ~ 5050 1650
+Wire Wire Line
+	5050 1650 5150 1650
 $EndSCHEMATC

Commit message: adding power facilities
Parts:
- R4: value 470R -> 670R
Connections:
- net +5V: now also R4.2
- net GND: no longer U2.2
- net HEATER: now also U2.2; no longer R4.2
Other:
- note added: "HEATER is active LOW"
Changed lines of the file:
@@
 	1900 3800 4400 3800
 Connection ~ 1900 1950
-Text GLabel 2650 4150 0    50   Input ~ 0
+Text GLabel 3000 4350 0    50   Input ~ 0
 HEATER
 $Comp
@@
 P 3000 4150
 F 0 "R4" V 2793 4150 50  0000 C CNN
-F 1 "470R" V 2884 4150 50  0000 C CNN
+F 1 "670R" V 2884 4150 50  0000 C CNN
 F 2 "" V 2930 4150 50  0001 C CNN
 F 3 "~" H 3000 4150 50  0001 C CNN
@@
 	0    1    1    0
 $EndComp
-$Comp
-L power:GND #PWR05
-U 1 1 62E3B65A
-P 3150 4450
-F 0 "#PWR05" H 3150 4200 50  0001 C CNN
-F 1 "GND" H 3155 4277 50  0000 C CNN
-F 2 "" H 3150 4450 50  0001 C CNN
-F 3 "" H 3150 4450 50  0001 C CNN
-	1    3150 4450
-	1    0    0    -1
-$EndComp
 Wire Wire Line
 	2650 4150 2850 4150
 Wire Wire Line
 	3150 4150 3350 4150
-Wire Wire Line
-	3350 4350 3150 4350
-Wire Wire Line
-	3150 4350 3150 4450
 Wire Wire Line
 	4400 4150 4400 3800
@@
 Wire Wire Line
 	5050 1650 5150 1650
+$Comp
+L power:+5V #PWR?
+U 1 1 62EC4FF6
+P 2650 4150
+F 0 "#PWR?" H 2650 4000 50  0001 C CNN
+F 1 "+5V" H 2665 4323 50  0000 C CNN
+F 2 "" H 2650 4150 50  0001 C CNN
+F 3 "" H 2650 4150 50  0001 C CNN
+	1    2650 4150
+	1    0    0    -1
+$EndComp
+Wire Wire Line
+	3350 4350 3000 4350
+Text Notes 2700 4550 0    50   ~ 0
+HEATER is active LOW
 $EndSCHEMATC
